Commit message: so_arm_100_description: move files to so_arm_100_description
Signed-off-by: Rhys Mainwaring <rhys.mainwaring@me.com>

File: so_arm_100_description/urdf/so_arm_100.urdf (robot description, URDF)
Before this commit: robot so_100_arm, 8 links, 7 joints
Links:
- link Base: geometry collision mesh filename=package://so_arm_100_moveit_config/models/so_arm_100_5dof/m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; visual mesh filename=package://so_arm_100_moveit_config/models/so_arm_100_5dof/m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
- link Fixed_Gripper: geometry collision mesh filename=package://so_arm_100_moveit_config/models/so_arm_100_5dof/m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; visual mesh filename=package://so_arm_100_moveit_config/models/so_arm_100_5dof/m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
- link Lower_Arm: geometry collision mesh filename=package://so_arm_100_moveit_config/models/so_arm_100_5dof/m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; visual mesh filename=package://so_arm_100_moveit_config/models/so_arm_100_5dof/m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
- link Moving_Jaw: geometry collision mesh filename=package://so_arm_100_moveit_config/models/so_arm_100_5dof/m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; visual mesh filename=package://so_arm_100_moveit_config/models/so_arm_100_5dof/m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
- link Shoulder_Rotation_Pitch: geometry collision mesh filename=package://so_arm_100_moveit_config/models/so_arm_100_5dof/m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; visual mesh filename=package://so_arm_100_moveit_config/models/so_arm_100_5dof/m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
- link Upper_Arm: geometry collision mesh filename=package://so_arm_100_moveit_config/models/so_arm_100_5dof/m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; visual mesh filename=package://so_arm_100_moveit_config/models/so_arm_100_5dof/m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
- link Wrist_Pitch_Roll: geometry collision mesh filename=package://so_arm_100_moveit_config/models/so_arm_100_5dof/m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; visual mesh filename=package://so_arm_100_moveit_config/models/so_arm_100_5dof/m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

File: so_arm_100_description/urdf/so_arm_100_5dof.urdf (robot description, URDF)
Before this commit: robot so_100_arm, 8 links, 7 joints
Links:
- link Base: geometry collision mesh filename=package://so_arm_100_moveit_config/models/so_arm_100_5dof/m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; visual mesh filename=package://so_arm_100_moveit_config/models/so_arm_100_5dof/m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
- link Fixed_Gripper: geometry collision mesh filename=package://so_arm_100_moveit_config/models/so_arm_100_5dof/m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; visual mesh filename=package://so_arm_100_moveit_config/models/so_arm_100_5dof/m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
- link Lower_Arm: geometry collision mesh filename=package://so_arm_100_moveit_config/models/so_arm_100_5dof/m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; visual mesh filename=package://so_arm_100_moveit_config/models/so_arm_100_5dof/m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
- link Moving_Jaw: geometry collision mesh filename=package://so_arm_100_moveit_config/models/so_arm_100_5dof/m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; visual mesh filename=package://so_arm_100_moveit_config/models/so_arm_100_5dof/m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
- link Shoulder_Rotation_Pitch: geometry collision mesh filename=package://so_arm_100_moveit_config/models/so_arm_100_5dof/m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; visual mesh filename=package://so_arm_100_moveit_config/models/so_arm_100_5dof/m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
- link Upper_Arm: geometry collision mesh filename=package://so_arm_100_moveit_config/models/so_arm_100_5dof/m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; visual mesh filename=package://so_arm_100_moveit_config/models/so_arm_100_5dof/m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
- link Wrist_Pitch_Roll: geometry collision mesh filename=package://so_arm_100_moveit_config/models/so_arm_100_5dof/m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; visual mesh filename=package://so_arm_100_moveit_config/models/so_arm_100_5dof/m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

File: so_arm_100_description/urdf/so_arm_100_5dof_hardware.urdf (robot description, URDF)
Before this commit: robot so_100_arm, 8 links, 7 joints
Links:
- link Base: geometry collision mesh filename=file://$(find so_arm_100_moveit_config)/models/so_arm_100_5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; visual mesh filename=file://$(find so_arm_100_moveit_config)/models/so_arm_100_5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
- link Fixed_Gripper: geometry collision mesh filename=file://$(find so_arm_100_moveit_config)/models/so_arm_100_5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 scale=0.9 0.9 0.9; visual mesh filename=file://$(find so_arm_100_moveit_config)/models/so_arm_100_5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
- link Lower_Arm: geometry collision mesh filename=file://$(find so_arm_100_moveit_config)/models/so_arm_100_5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 scale=0.9 0.9 0.9; visual mesh filename=file://$(find so_arm_100_moveit_config)/models/so_arm_100_5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
- link Moving_Jaw: geometry collision mesh filename=file://$(find so_arm_100_moveit_config)/models/so_arm_100_5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 scale=0.9 0.9 0.9; visual mesh filename=file://$(find so_arm_100_moveit_config)/models/so_arm_100_5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
- link Shoulder_Rotation_Pitch: geometry collision mesh filename=file://$(find so_arm_100_moveit_config)/models/so_arm_100_5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 scale=0.9 0.9 0.9; visual mesh filename=file://$(find so_arm_100_moveit_config)/models/so_arm_100_5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
- link Upper_Arm: geometry collision mesh filename=file://$(find so_arm_100_moveit_config)/models/so_arm_100_5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 scale=0.9 0.9 0.9; visual mesh filename=file://$(find so_arm_100_moveit_config)/models/so_arm_100_5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
- link Wrist_Pitch_Roll: geometry collision mesh filename=file://$(find so_arm_100_moveit_config)/models/so_arm_100_5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 scale=0.9 0.9 0.9; visual mesh filename=file://$(find so_arm_100_moveit_config)/models/so_arm_100_5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
