Commit message: Vendor so_arm_100_hardware and make this fork self-contained
- Vendor the so_arm_100_hardware driver into this repo (was a separate
  brukg/so_arm_100_hardware repo). Its source now targets the Humble
  ros2_control API directly, so no build-time compat patch is needed.
- Bake this machine's serial by-id path as the default everywhere,
  replacing /dev/ttyUSB0 (override with serial_port:=...).
- Load config/calibration.yaml by default in hardware.launch.py; zero_ticks
  measured from the physical home pose, plus optional per-joint
  gravity_coefficient feedforward to counter droop when extended.
- Add real goal/trajectory constraints to the arm_controller so missed
  targets report ABORTED instead of a false SUCCEEDED.
- Wire calibration_file through the xacro -> ros2_control hardware params.
- Rewrite README for the single-repo, no-patch workflow.

Co-Authored-By: Claude Opus 4.8 <noreply@anthropic.com>

File: so_arm_100_description/ros2_control/so_arm_100_5dof_position.ros2_control.xacro (robot description, xacro)
@@ -9,5 +9,5 @@
       use_topic_hardware_interface:=^|false
       use_fake_hardware:=^|false
-      serial_port:=^|/dev/ttyUSB0
+      serial_port:=^|/dev/serial/by-id/usb-1a86_USB_Single_Serial_5970073059-if00
       serial_baudrate:=^|1000000
       servo_speed:=^|2400

File: so_arm_100_moveit_config/config/so_arm_100.ros2_control.xacro (robot description, xacro)
@@ -1,5 +1,5 @@
 <?xml version="1.0"?>
 <robot xmlns:xacro="http://www.ros.org/wiki/xacro">
-    <xacro:macro name="so_arm_100_ros2_control" params="name initial_positions_file use_fake_hardware serial_port:=^|/dev/ttyUSB0 serial_baudrate:=^|1000000 servo_speed:=^|2400 servo_acceleration:=^|50" >
+    <xacro:macro name="so_arm_100_ros2_control" params="name initial_positions_file use_fake_hardware serial_port:=^|/dev/serial/by-id/usb-1a86_USB_Single_Serial_5970073059-if00 serial_baudrate:=^|1000000 servo_speed:=^|2400 servo_acceleration:=^|50 calibration_file:=^|''" >
         <xacro:property name="initial_positions" value="${xacro.load_yaml(initial_positions_file)['initial_positions']}"/>
         <ros2_control name="${name}" type="system">
@@ -15,4 +15,7 @@
                     <param name="servo_speed">${servo_speed}</param>
                     <param name="servo_acceleration">${servo_acceleration}</param>
+                    <xacro:if value="${calibration_file != ''}">
+                      <param name="calibration_file">${calibration_file}</param>
+                    </xacro:if>
                 </xacro:unless>
             </hardware>

File: so_arm_100_moveit_config/config/so_arm_100.urdf.xacro (robot description, xacro)
@@ -4,5 +4,6 @@
     <xacro:arg name="initial_positions_file" default="initial_positions.yaml" />
     <xacro:arg name="use_fake_hardware" default="false"/>
-    <xacro:arg name="serial_port" default="/dev/ttyUSB0"/>
+    <xacro:arg name="serial_port" default="/dev/serial/by-id/usb-1a86_USB_Single_Serial_5970073059-if00"/>
+    <xacro:arg name="calibration_file" default=""/>
     <xacro:arg name="serial_baudrate" default="1000000"/>
     <xacro:arg name="servo_speed" default="2400"/>
@@ -18,4 +19,5 @@
         use_fake_hardware="$(arg use_fake_hardware)"
         serial_port="$(arg serial_port)"
+        calibration_file="$(arg calibration_file)"
         serial_baudrate="$(arg serial_baudrate)"
         servo_speed="$(arg servo_speed)"
