Commit message: build process with build file

File: so_arm_100_description/ros2_control/so_arm_100_5dof_position.ros2_control.xacro (robot description, xacro)
@@ -121,6 +121,10 @@
       </joint>
       <joint name="${prefix}Gripper">
+        <!-- min widened 2026-08-02 to stay consistent with
+             so_arm_100_5dof_arm.urdf.xacro's Gripper joint limit (see that
+             file's comment for why, and for which launch paths actually
+             use this file vs. moveit_config's own ros2_control.xacro). -->
         <command_interface name="position">
-          <param name="min">-0.1792</param>
+          <param name="min">-0.24</param>
           <param name="max">1.57</param>
           <xacro:if value="${initial_positions_file != ''}">

File: so_arm_100_description/urdf/so_arm_100_5dof_arm.urdf.xacro (robot description, xacro)
@@ -404,5 +404,19 @@
     <axis
       xyz="0 0 1" />
-    <limit effort="1000" lower="-0.1792" upper="1.5708" velocity="5.0"/>
+    <!-- lower widened 2026-08-02 (-0.1792 to -0.24 rad, ~-13.75deg): -12deg
+         grasp closes are already hardware-proven, and -0.1792 (~-10.27deg)
+         was blocking tune_grasp from testing -11/-12/-13deg at all. Kept a
+         deliberately small ~0.75deg margin past -13deg, not a big jump.
+         This IS the real bound for real hardware: pickandplace_demo.launch.py
+         and hardware.launch.py both build robot_description from
+         so_arm_100_moveit_config/config/so_arm_100.urdf.xacro (which
+         includes this file), whose own ros2_control.xacro declares no
+         min/max at all for any joint, so MoveIt/OMPL's use of this <limit>
+         is the only enforced bound. so_arm_100_description's own
+         ros2_control.xacro (a separate file, also has a Gripper min, kept
+         in sync here) is NOT part of that chain, it's only reachable via
+         so_arm_100_5dof.urdf.xacro, the description package's standalone
+         display/demo entry point, unused by real hardware runs today. -->
+    <limit effort="1000" lower="-0.24" upper="1.5708" velocity="5.0"/>
     <dynamics damping="0.1"/>
   </joint>
